File: KiCad Files/NextGen Macropad/NextGen Macropad.kicad_pcb (KiCad board)
At the start: 2 copper layers, 80.4 x 119.2 mm, 80 parts, among them J1 OLED_128x64, J2 Battery JST-PH, J3 USB_C_Receptacle_USB2.0_16P, Q1 AO3401A, SW1 SW_Push_45deg, SW10 SW_Push_45deg, SW11 SW_Push_45deg, SW12 SW_Push_45deg, SW13 SW_Push_45deg, SW14 SW_Push_45deg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

Commit message: Uploading KiCad + Images + Production 180326-1005
Routing:
- net (no net): track 0.23 -> 0.00 mm, vias 85 -> 1
- net GND: vias 14 -> 98
- added copper zone on B.Cu, net GND
- added copper zone on F.Cu, net GND
- removed copper zone on B.Cu, net (none)
- removed copper zone on F.Cu, net (none)
