File: KiCad Files/NextGen Macropad/NextGen Macropad.kicad_pcb (KiCad board)
At the start: 2 copper layers, 80.4 x 119.2 mm, 80 parts, among them J1 OLED_128x64, J2 Battery JST-PH, J3 USB_C_Receptacle_USB2.0_16P, Q1 AO3401A, SW1 SW_Push_45deg, SW10 SW_Push_45deg, SW11 SW_Push_45deg, SW12 SW_Push_45deg, SW13 SW_Push_45deg, SW14 SW_Push_45deg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

Commit message: Fix PCB + Add BOM
Parts:
- C1, C2, C4, C5, D17, D18, D33, Q1, R1, R2, R3, R8, U2, U3: moved to B.Cu
- turned C5 to 0 degrees
- turned D17 to 180 degrees
- turned D18 to 180 degrees
- turned Q1 to 180 degrees
- turned R2 to 0 degrees
- turned R3 to 0 degrees
- turned U2 to 180 degrees
- turned U3 to 0 degrees
- renumbered Reset to SW18, Boot to SW19
Routing:
- net GND: track 627.5 -> 565.3 mm, vias 98 -> 134
- net Net-(U2-~{CHRG}): track 28.7 -> 46.8 mm
- net /REG - EN: track 190.5 -> 208.1 mm, vias 3 -> 4
- net Net-(U2-~{STDBY}): track 31.3 -> 47.6 mm
- net Net-(U2-PROG): track 2.42 -> 14.3 mm, vias 0 -> 2
- net /LED DIN: track 50.2 -> 41.4 mm
- net /ROW 3: track 145.3 -> 137.4 mm
- net /B +: track 51.3 -> 58.8 mm, vias 1 -> 2
- net Net-(L14-DOUT): track 14.6 -> 20.8 mm
- net Net-(D17-Pad2): track 1.75 -> 7.38 mm
- net Net-(D18-Pad2): track 1.75 -> 7.37 mm
- net Net-(L6-DOUT): track 15.3 -> 20.8 mm
- net /MOSFET: track 197.0 -> 202.1 mm, vias 4 -> 6
- net /COLO 3: track 191.9 -> 187.3 mm
- net Net-(L15-DOUT): track 16.1 -> 19.6 mm
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Other:
- board size 80.4 x 119.2 mm -> 80.4 x 119.4 mm

Commit message: New PCB Layout
Parts:
- added G***: LOGO, Dragon Emblem:White DevX Official Logo, F.Cu at (89.8, 60.4)
- added G***: LOGO, Dragon Emblem:White DevX Official Logo, B.Cu at (141.7, 58.7)
- D1, D10, D11, D12, D13, D14, D15, D16, D2, D3, D4, D5, D6, D7, D8, D9: footprint ScottoKeebs_Components:Diode_DO-35 -> ScottoKeebs_Components:Diode_SOD-123
- R10, R13, R14, R9: moved to B.Cu
- SW18, SW19: footprint Button_Switch_SMD:SW_Push_1TS009xxxx-xxxx-xxxx_6x6x5mm -> Button_Switch_THT:SW_PUSH_6mm
- moved D1 7.48 mm to (97.0, 83.5), turned to 90 degrees
- moved D6 7.30 mm to (116.2, 102.5), turned to 90 degrees
- moved D13 7.27 mm to (154.2, 83.5), turned to 90 degrees
- moved D9 7.24 mm to (135.2, 83.5), turned to 90 degrees
- moved D16 7.22 mm to (154.2, 140.5), turned to 90 degrees
- moved D5 7.20 mm to (116.2, 83.5), turned to 90 degrees
- moved D10 7.19 mm to (135.2, 102.5), turned to 90 degrees
- moved D14 7.19 mm to (154.2, 102.5), turned to 90 degrees
- moved D15 7.19 mm to (154.2, 121.5), turned to 90 degrees
- moved D12 7.15 mm to (135.2, 140.5), turned to 90 degrees
- moved D11 7.15 mm to (135.2, 121.5), turned to 90 degrees
- moved D7 7.10 mm to (116.1, 121.5), turned to 90 degrees
- moved D4 7.08 mm to (97.1, 140.5), turned to 90 degrees
- moved D3 7.06 mm to (97.0, 121.5), turned to 90 degrees
- moved D2 7.05 mm to (97.0, 102.5), turned to 90 degrees
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Routing:
- net GND: track 565.3 -> 129.4 mm, vias 134 -> 86
- net /COLO 3: track 187.3 -> 137.7 mm, vias 2 -> 7
- net /REG - EN: track 208.1 -> 161.4 mm
- net /VOLT-DIV: track 173.7 -> 131.5 mm, vias 6 -> 4
- net /COLO 1: track 143.5 -> 103.0 mm, vias 1 -> 7
- net /COLO 2: track 157.7 -> 120.0 mm, vias 2 -> 7
- net /COLO 0: track 118.2 -> 82.0 mm
- net +5V: track 551.0 -> 583.8 mm, vias 14 -> 32
- net /MOSFET: track 202.1 -> 181.6 mm
- net /RESET PIN: track 10.1 -> 22.9 mm, vias 0 -> 1
- net /ROW 2: track 121.9 -> 110.6 mm, vias 6 -> 2
- net /Boot: track 28.1 -> 38.5 mm, vias 0 -> 2
- net /ROW 1: track 131.1 -> 121.1 mm, vias 6 -> 2
- net +3.3V: track 221.9 -> 212.1 mm, vias 3 -> 2
- net Net-(U2-~{STDBY}): track 47.6 -> 56.6 mm, vias 2 -> 4
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Other:
- board size 80.4 x 119.4 mm -> 80.4 x 120 mm
- board text added: "+"
- board text added: "-"

Commit message: KiCad Change
Parts:
- added ?: , , F.Cu at (78.0, 161.3)
- added ?: , , F.Cu at (154.4, 161.2)
- added kibuzzard-69BEA4AE: G***, kibuzzard-69BEA4AE, F.Cu at (150.8, 153.0)
Other:
- board text added: "Powered by DevX-Dragon"
