File: KiCad Files/NextGen Macropad/NextGen Macropad.kicad_sch (KiCad schematic)
At the start: 80 parts, among them J1 OLED_128x64, J2 Battery JST-PH, J3 USB_C_Receptacle_USB2.0_16P, Q1 AO3401A, SW1 SW_Push_45deg, SW10 SW_Push_45deg, SW11 SW_Push_45deg, SW12 SW_Push_45deg, SW13 SW_Push_45deg, SW14 SW_Push_45deg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

Commit message: Uploading KiCad + Images + Production 180326-1005
Changed lines of the file:
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@@
 	)
 	(junction
-		(at 223.52 139.7)
-		(diameter 0)
-		(color 0 0 0 0)
-	)
-	(junction
 		(at 52.07 143.51)
 		(diameter 0)
@@
 	)
 	(junction
+		(at 224.79 152.4)
+		(diameter 0)
+		(color 0 0 0 0)
+	)
+	(junction
 		(at 24.13 100.33)
 		(diameter 0)
@@
 	)
 	(junction
+		(at 223.52 139.7)
+		(diameter 0)
+		(color 0 0 0 0)
+	)
+	(junction
 		(at 24.13 130.81)
 		(diameter 0)
@@
 	)
 	(junction
-		(at 224.79 153.67)
-		(diameter 0)
-		(color 0 0 0 0)
-	)
-	(junction
 		(at 46.99 115.57)
 		(diameter 0)
@@
 	(wire
 		(pts
+			(xy 228.6 152.4) (xy 228.6 153.67)
+		)
+		(stroke
+			(width 0)
+			(type default)
+		)
+	)
+	(wire
+		(pts
 			(xy 275.59 130.81) (xy 271.78 130.81)
 		)
@@
 	(wire
 		(pts
-			(xy 223.52 139.7) (xy 226.06 139.7)
-		)
-		(stroke
-			(width 0)
-			(type default)
-		)
-	)
-	(wire
-		(pts
 			(xy 224.79 162.56) (xy 210.82 162.56)
 		)
@@
 	(wire
 		(pts
-			(xy 224.79 153.67) (xy 224.79 162.56)
+			(xy 226.06 138.43) (xy 226.06 139.7)
 		)
 		(stroke
@@
 	(wire
 		(pts
+			(xy 223.52 139.7) (xy 223.52 147.32)
+		)
+		(stroke
+			(width 0)
+			(type default)
+		)
+	)
+	(wire
+		(pts
 			(xy 172.72 43.18) (xy 182.88 43.18)
 		)
@@
 	(wire
 		(pts
-			(xy 223.52 128.27) (xy 223.52 139.7)
-		)
-		(stroke
-			(width 0)
-			(type default)
-		)
-	)
-	(wire
-		(pts
 			(xy 177.8 147.32) (xy 194.31 147.32)
 		)
@@
 	(wire
 		(pts
+			(xy 224.79 152.4) (xy 224.79 162.56)
+		)
+		(stroke
+			(width 0)
+			(type default)
+		)
+	)
+	(wire
+		(pts
 			(xy 210.82 147.32) (xy 223.52 147.32)
 		)
@@
 	(wire
 		(pts
-			(xy 224.79 143.51) (xy 224.79 153.67)
+			(xy 224.79 143.51) (xy 224.79 152.4)
 		)
 		(stroke
@@
 	(wire
 		(pts
-			(xy 224.79 153.67) (xy 227.33 153.67)
+			(xy 129.54 87.63) (xy 137.16 87.63)
 		)
 		(stroke
@@
 	(wire
 		(pts
-			(xy 129.54 87.63) (xy 137.16 87.63)
+			(xy 166.37 81.28) (xy 161.29 81.28)
 		)
 		(stroke
@@
 	(wire
 		(pts
-			(xy 166.37 81.28) (xy 161.29 81.28)
+			(xy 24.13 87.63) (xy 24.13 100.33)
 		)
 		(stroke
@@
 	(wire
 		(pts
-			(xy 24.13 87.63) (xy 24.13 100.33)
+			(xy 95.25 143.51) (xy 111.76 143.51)
 		)
 		(stroke
@@
 	(wire
 		(pts
-			(xy 95.25 143.51) (xy 111.76 143.51)
+			(xy 152.4 69.85) (xy 166.37 69.85)
 		)
 		(stroke
@@
 	(wire
 		(pts
-			(xy 152.4 69.85) (xy 166.37 69.85)
+			(xy 223.52 128.27) (xy 223.52 139.7)
 		)
 		(stroke
@@
 	(wire
 		(pts
+			(xy 226.06 139.7) (xy 223.52 139.7)
+		)
+		(stroke
+			(width 0)
+			(type default)
+		)
+	)
+	(wire
+		(pts
 			(xy 198.12 34.29) (xy 196.85 34.29)
 		)
@@
 	(wire
 		(pts
-			(xy 168.91 154.94) (xy 170.18 154.94)
+			(xy 224.79 152.4) (xy 228.6 152.4)
 		)
 		(stroke
@@
 	(wire
 		(pts
-			(xy 111.76 162.56) (xy 128.27 162.56)
+			(xy 168.91 154.94) (xy 170.18 154.94)
 		)
 		(stroke
@@
 	(wire
 		(pts
-			(xy 175.26 80.01) (xy 185.42 80.01)
+			(xy 111.76 162.56) (xy 128.27 162.56)
 		)
 		(stroke
@@
 	(wire
 		(pts
-			(xy 266.7 38.1) (xy 267.97 38.1)
+			(xy 175.26 80.01) (xy 185.42 80.01)
 		)
 		(stroke
@@
 	(wire
 		(pts
-			(xy 266.7 46.99) (xy 266.7 48.26)
+			(xy 266.7 38.1) (xy 267.97 38.1)
 		)
 		(stroke
@@
 	(wire
 		(pts
-			(xy 223.52 147.32) (xy 223.52 139.7)
+			(xy 266.7 46.99) (xy 266.7 48.26)
 		)
 		(stroke
@@
 	(symbol
 		(lib_id "power:+5V")
-		(at 226.06 139.7 0)
+		(at 226.06 138.43 0)
 		(unit 1)
 		(exclude_from_sim no)
@@
 		(fields_autoplaced yes)
 		(property "Reference" "#PWR01"
-			(at 226.06 143.51 0)
+			(at 226.06 142.24 0)
 			(effects
 				(font
@@
 		)
 		(property "Value" "+5V"
-			(at 226.06 134.62 0)
+			(at 226.06 133.35 0)
 			(effects
 				(font
@@
 		)
 		(property "Footprint" ""
-			(at 226.06 139.7 0)
+			(at 226.06 138.43 0)
 			(effects
 				(font
@@
 		)
 		(property "Datasheet" ""
-			(at 226.06 139.7 0)
+			(at 226.06 138.43 0)
 			(effects
 				(font
@@
 		)
 		(property "Description" "Power symbol creates a global label with name \"+5V\""
-			(at 226.06 139.7 0)
+			(at 226.06 138.43 0)
 			(effects
 				(font
@@
 	(symbol
 		(lib_id "power:GND")
-		(at 227.33 153.67 0)
+		(at 228.6 153.67 0)
 		(unit 1)
 		(exclude_from_sim no)
@@
 		(fields_autoplaced yes)
 		(property "Reference" "#PWR02"
-			(at 227.33 160.02 0)
+			(at 228.6 160.02 0)
 			(effects
 				(font
@@
 		)
 		(property "Value" "GND"
-			(at 227.33 158.75 0)
+			(at 228.6 158.75 0)
 			(effects
 				(font
@@
 		)
 		(property "Footprint" ""
-			(at 227.33 153.67 0)
+			(at 228.6 153.67 0)
 			(effects
 				(font
@@
 		)
 		(property "Datasheet" ""
-			(at 227.33 153.67 0)
+			(at 228.6 153.67 0)
 			(effects
 				(font
@@
 		)
 		(property "Description" "Power symbol creates a global label with name \"GND\" , ground"
-			(at 227.33 153.67 0)
+			(at 228.6 153.67 0)
 			(effects
 				(font

Commit message: Fix PCB + Add BOM
Parts:
- D17, D18: LCSC (none) -> C2298
- J3: LCSC (none) -> C165948
- SW18, SW19: LCSC (none) -> C42416254
- U2: LCSC (none) -> C16581
- U3: LCSC (none) -> C23380830
Changed lines of the file:
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@@
 			)
 		)
+		(property "LCSC" "C16581"
+			(at 116.84 104.14 0)
+			(effects
+				(font
+					(size 1.27 1.27)
+				)
+				(hide yes)
+			)
+		)
 		(pin "3"
 		)
@@
 			)
 		)
+		(property "LCSC" "C42416254"
+			(at 128.27 21.59 0)
+			(effects
+				(font
+					(size 1.27 1.27)
+				)
+				(hide yes)
+			)
+		)
 		(pin "2"
 		)
@@
 			)
 		)
+		(property "LCSC" "C2298"
+			(at 100.33 104.14 0)
+			(effects
+				(font
+					(size 1.27 1.27)
+				)
+				(hide yes)
+			)
+		)
 		(pin "2"
 		)
@@
 			)
 		)
+		(property "LCSC" "C42416254"
+			(at 128.27 26.67 0)
+			(effects
+				(font
+					(size 1.27 1.27)
+				)
+				(hide yes)
+			)
+		)
 		(pin "2"
 		)
@@
 			)
 		)
+		(property "LCSC" "C23380830"
+			(at 45.72 31.75 0)
+			(effects
+				(font
+					(size 1.27 1.27)
+				)
+				(hide yes)
+			)
+		)
 		(pin "3"
 		)
@@
 			)
 		)
+		(property "LCSC" "C165948"
+			(at 251.46 48.26 0)
+			(effects
+				(font
+					(size 1.27 1.27)
+				)
+				(hide yes)
+			)
+		)
 		(pin "B4"
 		)
@@
 			(at 100.33 107.95 0)
 			(effects
+				(font
+					(size 1.27 1.27)
+				)
+				(hide yes)
+			)
+		)
+		(property "LCSC" "C2298"
+			(at 100.33 107.95 0)
+			(effects
